Commit message: Add the klara package with arm kinematics, plus base_link and tcp_L frames
klara.kinematics reads an arm's chain from the URDF and solves inverse
kinematics with damped least squares. It supports the five things a
5-joint arm can control: tool position, pitch (asin of the approach
direction's vertical part) and roll (measured from the arm's own
bending axis). Both angles come from the arm, not the target
position, because the bending plane sits ~3 cm off the base's yaw
axis.

Searches start from the seed, then from candidates with the base
already turned to face the target. Joints pinned at a limit drop out
of the step. Arm.line() plans a straight line, seeding every waypoint
from the last and reporting how far along it got when it can't
finish.

FK matches robot_state_publisher exactly at the home pose.

The URDF gains base_link (on the floor under the cart's center, x
toward the robot's front, since the original root faces backward) and
tcp_L (between the left fingertips, drawn as a red sphere). RViz shows
the base_link axes.

Co-Authored-By: Claude Opus 5.5 <noreply@anthropic.com>

File: ros2_ws/src/xlerobot_description/urdf/xlerobot.urdf (robot description, URDF)
Before this commit: robot xlerobot, 41 links, 40 joints
Links:
- added link base_link
- added link tcp_L; visual sphere radius=0.005
Joints:
- added joint base_link_joint: type fixed, parent world, child base_link, origin xyz=0 0 0 rpy=0 0 3.1415927
- added joint tcp_L_joint: type fixed, parent Fixed_Jaw, child tcp_L, origin xyz=0.008 -0.090 0 rpy=1.5707963 0 0
